File: Dice2.kicad_sch (KiCad schematic)
At the start: 23 parts, among them IC3 CD4511BE, U17 ULN2803A, U6 NE555P, U7 CD4029BE

Commit message: stuff
Parts:
- removed S3: B3F-1000, SamacSys_Parts:B3F4050, symbol dk_Tactile-Switches:B3F-1000
- added J12: DICE2, Connector_Wire:SolderWire-0.5sqmm_1x02_P4.6mm_D0.9mm_OD2.1mm, symbol Connector_Generic:Conn_01x02
Connections:
- net +5V: now also J12.1 (Pin_1)
- net D2Set: now also J12.2 (Pin_2)
Changed lines of the file:
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@@
+    (stroke (width 0) (type default) (color 0 0 0 0))
+  )
+  (wire (pts (xy 55.88 152.4) (xy 55.88 149.86))
     (stroke (width 0) (type default) (color 0 0 0 0))
   )
@@
     (stroke (width 0) (type default) (color 0 0 0 0))
   )
-  (wire (pts (xy 58.42 152.4) (xy 64.77 152.4))
+  (wire (pts (xy 55.88 152.4) (xy 64.77 152.4))
     (stroke (width 0) (type default) (color 0 0 0 0))
   )
@@
     (stroke (width 0) (type default) (color 0 0 0 0))
   )
+  (wire (pts (xy 53.34 149.86) (xy 53.34 152.4))
+    (stroke (width 0) (type default) (color 0 0 0 0))
+  )
   (wire (pts (xy 49.53 76.2) (xy 49.53 78.74))
     (stroke (width 0) (type default) (color 0 0 0 0))
   )
-  (wire (pts (xy 39.37 152.4) (xy 48.26 152.4))
+  (wire (pts (xy 39.37 152.4) (xy 53.34 152.4))
     (stroke (width 0) (type default) (color 0 0 0 0))
   )
@@
     )
     (pin "1")
-  )
-  (symbol (lib_id "dk_Tactile-Switches:B3F-1000") (at 53.34 154.94 0) (unit 1)
-    (in_bom yes) (on_board yes) (fields_autoplaced)
-    (property "Reference" "S3" (id 0) (at 53.34 146.05 0)
-      (effects (font (size 1.524 1.524)))
-    )
-    (property "Value" "B3F-1000" (id 1) (at 53.34 149.86 0)
-      (effects (font (size 1.524 1.524)))
-    )
-    (property "Footprint" "SamacSys_Parts:B3F4050" (id 2) (at 58.42 149.86 0)
-      (effects (font (size 1.524 1.524)) (justify left) hide)
-    )
-    (property "Datasheet" "https://omronfs.omron.com/en_US/ecb/products/pdf/en-b3f.pdf" (id 3) (at 58.42 147.32 0)
-      (effects (font (size 1.524 1.524)) (justify left) hide)
-    )
-    (property "Digi-Key_PN" "SW400-ND" (id 4) (at 58.42 144.78 0)
-      (effects (font (size 1.524 1.524)) (justify left) hide)
-    )
-    (property "MPN" "B3F-1000" (id 5) (at 58.42 142.24 0)
-      (effects (font (size 1.524 1.524)) (justify left) hide)
-    )
-    (property "Category" "Switches" (id 6) (at 58.42 139.7 0)
-      (effects (font (size 1.524 1.524)) (justify left) hide)
-    )
-    (property "Family" "Tactile Switches" (id 7) (at 58.42 137.16 0)
-      (effects (font (size 1.524 1.524)) (justify left) hide)
-    )
-    (property "DK_Datasheet_Link" "https://omronfs.omron.com/en_US/ecb/products/pdf/en-b3f.pdf" (id 8) (at 58.42 134.62 0)
-      (effects (font (size 1.524 1.524)) (justify left) hide)
-    )
-    (property "DK_Detail_Page" "/product-detail/en/omron-electronics-inc-emc-div/B3F-1000/SW400-ND/33150" (id 9) (at 58.42 132.08 0)
-      (effects (font (size 1.524 1.524)) (justify left) hide)
-    )
-    (property "Description" "SWITCH TACTILE SPST-NO 0.05A 24V" (id 10) (at 58.42 129.54 0)
-      (effects (font (size 1.524 1.524)) (justify left) hide)
-    )
-    (property "Manufacturer" "Omron Electronics Inc-EMC Div" (id 11) (at 58.42 127 0)
-      (effects (font (size 1.524 1.524)) (justify left) hide)
-    )
-    (property "Status" "Active" (id 12) (at 58.42 124.46 0)
-      (effects (font (size 1.524 1.524)) (justify left) hide)
-    )
-    (pin "1")
-    (pin "2")
-    (pin "3")
-    (pin "4")
   )
   (symbol (lib_id "power:+5V") (at 16.51 41.91 0) (unit 1)
@@
     )
     (pin "1")
+    (pin "2")
+  )
+  (symbol (lib_id "Connector_Generic:Conn_01x02") (at 53.34 144.78 90) (unit 1)
+    (in_bom yes) (on_board yes) (fields_autoplaced)
+    (property "Reference" "J12" (id 0) (at 58.42 143.5099 90)
+      (effects (font (size 1.27 1.27)) (justify right))
+    )
+    (property "Value" "DICE2" (id 1) (at 58.42 146.0499 90)
+      (effects (font (size 1.27 1.27)) (justify right))
+    )
+    (property "Footprint" "Connector_Wire:SolderWire-0.5sqmm_1x02_P4.6mm_D0.9mm_OD2.1mm" (id 2) (at 53.34 144.78 0)
+      (effects (font (size 1.27 1.27)) hide)
+    )
+    (property "Datasheet" "~" (id 3) (at 53.34 144.78 0)
+      (effects (font (size 1.27 1.27)) hide)
+    )
+    (pin "1")
