File: Dice3.kicad_sch (KiCad schematic)
At the start: 24 parts, among them IC4 CD4027BE, IC5 CD4511BE, U18 ULN2803A, U8 NE555P, U9 CD4029BE

Commit message: stuff
Parts:
- removed S4: B3F-4050, SamacSys_Parts:B3F4050, symbol dk_Tactile-Switches:B3F-1000
- added J13: DICE3, Connector_Wire:SolderWire-0.5sqmm_1x02_P4.6mm_D0.9mm_OD2.1mm, symbol Connector_Generic:Conn_01x02
Connections:
- net +5V: now also J13.1 (Pin_1)
- net at IC4.3 (CLOCK2), R12.1: now also J13.2 (Pin_2)
Changed lines of the file:
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@@
     (stroke (width 0) (type default) (color 0 0 0 0))
   )
-  (wire (pts (xy 34.29 152.4) (xy 40.64 152.4))
+  (wire (pts (xy 30.48 152.4) (xy 40.64 152.4))
     (stroke (width 0) (type default) (color 0 0 0 0))
   )
@@
     (stroke (width 0) (type default) (color 0 0 0 0))
   )
-  (wire (pts (xy 15.24 152.4) (xy 24.13 152.4))
+  (wire (pts (xy 15.24 152.4) (xy 27.94 152.4))
     (stroke (width 0) (type default) (color 0 0 0 0))
   )
@@
     (stroke (width 0) (type default) (color 0 0 0 0))
   )
+  (wire (pts (xy 30.48 149.86) (xy 30.48 152.4))
+    (stroke (width 0) (type default) (color 0 0 0 0))
+  )
   (wire (pts (xy 120.65 147.32) (xy 115.57 147.32))
     (stroke (width 0) (type default) (color 0 0 0 0))
@@
   )
   (wire (pts (xy 200.66 81.28) (xy 199.39 81.28))
+    (stroke (width 0) (type default) (color 0 0 0 0))
+  )
+  (wire (pts (xy 27.94 149.86) (xy 27.94 152.4))
     (stroke (width 0) (type default) (color 0 0 0 0))
   )
@@
     (pin "2")
   )
-  (symbol (lib_id "dk_Tactile-Switches:B3F-1000") (at 29.21 154.94 0) (unit 1)
-    (in_bom yes) (on_board yes) (fields_autoplaced)
-    (property "Reference" "S4" (id 0) (at 29.21 146.05 0)
-      (effects (font (size 1.524 1.524)))
-    )
-    (property "Value" "B3F-4050" (id 1) (at 29.21 149.86 0)
-      (effects (font (size 1.524 1.524)))
-    )
-    (property "Footprint" "SamacSys_Parts:B3F4050" (id 2) (at 34.29 149.86 0)
-      (effects (font (size 1.524 1.524)) (justify left) hide)
-    )
-    (property "Datasheet" "https://omronfs.omron.com/en_US/ecb/products/pdf/en-b3f.pdf" (id 3) (at 34.29 147.32 0)
-      (effects (font (size 1.524 1.524)) (justify left) hide)
-    )
-    (property "Digi-Key_PN" "SW400-ND" (id 4) (at 34.29 144.78 0)
-      (effects (font (size 1.524 1.524)) (justify left) hide)
-    )
-    (property "MPN" "B3F-1000" (id 5) (at 34.29 142.24 0)
-      (effects (font (size 1.524 1.524)) (justify left) hide)
-    )
-    (property "Category" "Switches" (id 6) (at 34.29 139.7 0)
-      (effects (font (size 1.524 1.524)) (justify left) hide)
-    )
-    (property "Family" "Tactile Switches" (id 7) (at 34.29 137.16 0)
-      (effects (font (size 1.524 1.524)) (justify left) hide)
-    )
-    (property "DK_Datasheet_Link" "https://omronfs.omron.com/en_US/ecb/products/pdf/en-b3f.pdf" (id 8) (at 34.29 134.62 0)
-      (effects (font (size 1.524 1.524)) (justify left) hide)
-    )
-    (property "DK_Detail_Page" "/product-detail/en/omron-electronics-inc-emc-div/B3F-1000/SW400-ND/33150" (id 9) (at 34.29 132.08 0)
-      (effects (font (size 1.524 1.524)) (justify left) hide)
-    )
-    (property "Description" "SWITCH TACTILE SPST-NO 0.05A 24V" (id 10) (at 34.29 129.54 0)
-      (effects (font (size 1.524 1.524)) (justify left) hide)
-    )
-    (property "Manufacturer" "Omron Electronics Inc-EMC Div" (id 11) (at 34.29 127 0)
-      (effects (font (size 1.524 1.524)) (justify left) hide)
-    )
-    (property "Status" "Active" (id 12) (at 34.29 124.46 0)
-      (effects (font (size 1.524 1.524)) (justify left) hide)
-    )
-    (pin "1")
-    (pin "2")
-    (pin "3")
-    (pin "4")
-  )
   (symbol (lib_id "power:+5V") (at 102.87 52.07 0) (unit 1)
     (in_bom yes) (on_board yes) (fields_autoplaced)
@@
     (pin "1")
   )
+  (symbol (lib_id "Connector_Generic:Conn_01x02") (at 27.94 144.78 90) (unit 1)
+    (in_bom yes) (on_board yes) (fields_autoplaced)
+    (property "Reference" "J13" (id 0) (at 33.02 143.5099 90)
+      (effects (font (size 1.27 1.27)) (justify right))
+    )
+    (property "Value" "DICE3" (id 1) (at 33.02 146.0499 90)
+      (effects (font (size 1.27 1.27)) (justify right))
+    )
+    (property "Footprint" "Connector_Wire:SolderWire-0.5sqmm_1x02_P4.6mm_D0.9mm_OD2.1mm" (id 2) (at 27.94 144.78 0)
+      (effects (font (size 1.27 1.27)) hide)
+    )
+    (property "Datasheet" "~" (id 3) (at 27.94 144.78 0)
+      (effects (font (size 1.27 1.27)) hide)
+    )
+    (pin "1")
+    (pin "2")
+  )
   (symbol (lib_id "Device:R") (at 247.65 45.72 90) (unit 1)
