File: Kniffel_V1.kicad_pcb (KiCad board)
At the start: 2 copper layers, 261.6 x 175.3 mm, 146 parts, among them IC1 CD4027BE, IC2 CD4511BE, IC3 CD4511BE, IC4 CD4027BE, IC5 CD4511BE, IC6 CD4511BE, IC7 CD4027BE, IC8 CD4511BE, J1 +9V, J2 GND, J3 USB 5V, J4 Switch, J5 5VOUT, J6 10VIN, U1 R-78HB5.0-0.5, U10 NE555P, U11 CD4029BE, U12 NE555P, U13 CD4029BE, U14 CD4093BE, U15 4017, U16 ULN2803A, U17 ULN2803A, U18 ULN2803A, U19 ULN2803A, U2 NE555P, U20 ULN2803A, U3 CD4029BE, U4 CD4093BE, U5 CD4093BE, U6 NE555P, U7 CD4029BE, U8 NE555P, U9 CD4029BE

Commit message: stuff
Parts:
- removed D19, D20, D21: LED, LED_THT:LED_D3.0mm
- removed G1, G2, G3, G4: MountingHole_3.2mm_M3, MountingHole:MountingHole_3.2mm_M3
- removed the R11 at (127.0, 132.1)
- removed the R16 at (172.7, 116.8)
- removed the R21 at (223.5, 134.6)
- removed the R26 at (281.9, 124.5)
- removed the R6 at (63.5, 132.1)
- added J10: ROLL_DICE, Connector_Wire:SolderWire-0.5sqmm_1x02_P4.6mm_D0.9mm_OD2.1mm, F.Cu at (86.8, 190.5)
- added J11: DICE1, Connector_Wire:SolderWire-0.5sqmm_1x02_P4.6mm_D0.9mm_OD2.1mm, F.Cu at (61.0, 121.9)
- added J12: DICE2, Connector_Wire:SolderWire-0.5sqmm_1x02_P4.6mm_D0.9mm_OD2.1mm, F.Cu at (61.0, 129.5)
- added J13: DICE3, Connector_Wire:SolderWire-0.5sqmm_1x02_P4.6mm_D0.9mm_OD2.1mm, F.Cu at (163.0, 121.9)
- added J14: DICE4, Connector_Wire:SolderWire-0.5sqmm_1x02_P4.6mm_D0.9mm_OD2.1mm, F.Cu at (162.6, 129.5)
- added J15: DICE5, Connector_Wire:SolderWire-0.5sqmm_1x02_P4.6mm_D0.9mm_OD2.1mm, F.Cu at (266.7, 134.6)
- added J16: RESET, Connector_Wire:SolderWire-0.5sqmm_1x02_P4.6mm_D0.9mm_OD2.1mm, F.Cu at (99.1, 190.5)
- added J7: LED1, Connector_Wire:SolderWire-0.5sqmm_1x02_P4.6mm_D0.9mm_OD2.1mm, F.Cu at (145.3, 188.0)
- added J8: LED2, Connector_Wire:SolderWire-0.5sqmm_1x02_P4.6mm_D0.9mm_OD2.1mm, F.Cu at (154.9, 188.0)
- added J9: LED3, Connector_Wire:SolderWire-0.5sqmm_1x02_P4.6mm_D0.9mm_OD2.1mm, F.Cu at (165.1, 188.0)
- R2: moved to F.Cu
- moved R7 198.3 mm to (83.8, 116.8), turned to 90 degrees
- moved J5 142.1 mm to (238.8, 182.9), turned to -90 degrees
- moved J6 140.5 mm to (246.4, 182.9), turned to -90 degrees
- moved R45 75.6 mm to (137.2, 116.8), turned to 90 degrees
- moved U19 71.2 mm to (201.9, 121.9)
- moved U20 69.0 mm to (252.7, 121.9)
- moved R65 66.8 mm to (276.9, 116.8), turned to 90 degrees
- moved R53 66.7 mm to (190.5, 116.8), turned to 90 degrees
- moved R57 66.6 mm to (228.6, 116.8), turned to 90 degrees
- moved R64 63.6 mm to (271.8, 116.8), turned to 90 degrees
- moved R55 63.3 mm to (218.4, 116.8), turned to 90 degrees
- moved R59 62.2 mm to (251.5, 116.8), turned to 90 degrees
- moved R60 62.0 mm to (238.8, 116.8), turned to 90 degrees
- moved R56 61.8 mm to (223.5, 116.8), turned to 90 degrees
- moved R42 61.2 mm to (144.8, 116.8)
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Routing:
- net GND: track 0.00 -> 939.9 mm
- net +5V: track 0.00 -> 865.9 mm
- net +10V: track 0.00 -> 573.9 mm
- net Reset: track 0.00 -> 326.0 mm, vias 0 -> 1
- net /Dice1/Roll: track 0.00 -> 192.5 mm
- net /Dice1/D4: track 0.00 -> 178.2 mm
- net /Dice1/D4Hold: track 0.00 -> 175.8 mm, vias 0 -> 1
- net /Dice1/D3Hold: track 0.00 -> 159.6 mm
- net /Dice1/D4Latch: track 0.00 -> 159.3 mm
- net /Dice1/D3: track 0.00 -> 124.1 mm
- net Net-(D14-Pad1): track 0.00 -> 122.4 mm
- net Net-(IC7-Pad3): track 0.00 -> 114.1 mm
- net /Dice1/D4R: track 0.00 -> 110.1 mm
- net /Dice1/D3Latch: track 0.00 -> 104.6 mm
- net Net-(IC7-Pad1): track 0.00 -> 88.9 mm, vias 0 -> 1
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
Commit message: changes
Parts:
- moved U4 26.9 mm to (33.0, 185.4), turned to 90 degrees
Routing:
- net GND: track 939.9 -> 991.2 mm
- net +10V: track 573.9 -> 607.5 mm
- net /Dice1/D2Latch: track 66.5 -> 94.3 mm
- net /Dice1/D2Hold: track 64.8 -> 89.9 mm, vias 1 -> 0
- net Net-(IC1-Pad3): track 86.8 -> 101.2 mm, vias 0 -> 1
- net +5V: track 865.9 -> 852.3 mm, vias 0 -> 1
- net /Dice1/D3Hold: track 159.6 -> 147.1 mm
- net /Dice1/D4Latch: track 159.3 -> 168.8 mm, vias 0 -> 1
- net Net-(IC4-Pad1): track 37.8 -> 46.4 mm
- net Net-(DS2-Pad4): track 16.9 -> 9.10 mm
- net Reset: track 326.0 -> 318.6 mm
- net Net-(U6-Pad3): track 35.7 -> 42.8 mm
- net Net-(D17-Pad2): track 76.3 -> 69.5 mm
- net /Dice1/D4Hold: track 175.8 -> 182.4 mm, vias 1 -> 0
- net Net-(DS2-Pad10): track 75.4 -> 69.0 mm
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
Commit message: final V1
Parts:
- added REF1: MountingHole_3.2mm_M3_DIN965_Pad, MountingHole:MountingHole_3.2mm_M3_DIN965_Pad, F.Cu at (34.0, 26.0)
- added REF2: MountingHole_3.2mm_M3_DIN965_Pad, MountingHole:MountingHole_3.2mm_M3_DIN965_Pad, F.Cu at (282.5, 26.5)
- added REF3: MountingHole_3.2mm_M3_DIN965_Pad, MountingHole:MountingHole_3.2mm_M3_DIN965_Pad, F.Cu at (283.5, 189.0)
- added REF4: MountingHole_3.2mm_M3_DIN965_Pad, MountingHole:MountingHole_3.2mm_M3_DIN965_Pad, F.Cu at (33.0, 191.0)
- J11, J12, J13, J14, J15: moved to B.Cu
- moved R12 14.7 mm to (169.6, 136.0), turned to 180 degrees
- moved J14 5.24 mm to (167.8, 129.5), turned to 180 degrees
- moved J11 5.08 mm to (66.0, 121.9), turned to 180 degrees
- moved J12 5.08 mm to (66.0, 129.5), turned to 180 degrees
- moved J13 4.36 mm to (167.4, 122.3), turned to 180 degrees
Routing:
- net (no net): track 0.00 -> 130.8 mm
- net GND: track 991.2 -> 928.0 mm
- net +10V: track 607.5 -> 563.4 mm
- net +5V: track 852.3 -> 820.0 mm, vias 1 -> 0
- net /Dice1/D3: track 123.2 -> 97.4 mm
- net /Dice1/D4Hold: track 182.4 -> 167.3 mm
- net Net-(IC1-Pad3): track 101.2 -> 86.2 mm, vias 1 -> 0
- net Net-(D2-Pad1): track 77.2 -> 92.1 mm
- net Net-(IC7-Pad1): track 88.3 -> 74.8 mm, vias 1 -> 0
- net Net-(D2-Pad2): track 41.4 -> 52.8 mm
- net Net-(IC4-Pad1): track 46.4 -> 37.2 mm
- net Net-(U2-Pad3): track 45.5 -> 36.4 mm
- net /Dice3/D4Set: track 51.5 -> 60.2 mm
- net /Dice1/D2: track 67.7 -> 60.5 mm
- net Net-(R60-Pad1): track 33.8 -> 41.0 mm
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Other:
- board text added: "Kniffel V1"
- board text added: "Maurizio Kerrutt"
- board text added: "Nico Brike"
- board text added: "Tobias Steinkamp"
- board text added: "Yannik Rattenholl"

Commit message: spelling :)
Other:
- board text added: "Nico Birke"
- board text removed: "Nico Brike"
Changed lines of the file:
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@@
     (effects (font (size 1 1) (thickness 0.15)) (justify left))
   )
-  (gr_text "Nico Brike" (at 111.5 134) (layer "F.SilkS")
+  (gr_text "Nico Birke" (at 111.5 134) (layer "F.SilkS")
     (effects (font (size 1 1) (thickness 0.15)) (justify left))
   )
